File: Letter_R.kicad_sch (KiCad schematic)
At the start: 19 parts, among them Q2 DMG2302UKQ-7, SW2 100SP1T1B4M2QE

Commit message: Add in changes: move to 0805 parts, routing updates
Parts:
- R14: footprint Custom_Parts:R_0402_1005Metric -> Custom_Parts:R_0805_2012Metric; symbol birthday:RC0402FR-07100KL -> birthday:RC0805FR-07100KL; MPN RC0402FR-07100KL -> RC0805FR-07100KL
Changed lines of the file:
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@@
 	)
 	(symbol
-		(lib_id "birthday:RC0402FR-07100KL")
+		(lib_id "birthday:RC0805FR-07100KL")
 		(at 177.8 78.74 180)
 		(unit 1)
@@
 			)
 		)
-		(property "Footprint" "Custom_Parts:R_0402_1005Metric"
+		(property "Footprint" "Custom_Parts:R_0805_2012Metric"
 			(at 177.8 78.74 0)
 			(hide yes)
@@
 			)
 		)
-		(property "Datasheet" "https://www.yageo.com/en/ProductSearch/PartNumberSearch?part_number=RC0402FR-07100KL"
+		(property "Datasheet" "https://www.yageo.com/en/ProductSearch/PartNumberSearch?part_number=RC0805FR-07100KL"
 			(at 177.8 78.74 0)
 			(hide yes)
@@
 			)
 		)
-		(property "Description" "Resistor, 100k, 1%, 62.5mW, 50V, 100ppm/C, Thick Film, 0402"
+		(property "Description" "Resistor, 100k, 1%, 125mW, 150V, 100ppm/C, Thick Film, 0805"
 			(at 177.8 78.74 0)
 			(hide yes)
@@
 			)
 		)
-		(property "MPN" "RC0402FR-07100KL"
+		(property "MPN" "RC0805FR-07100KL"
 			(at 177.8 78.74 0)
 			(hide yes)
