File: Griffin_kicad.kicad_pcb (KiCad board)
At the start: 2 copper layers, 212 x 66 mm, 127 parts, among them J1 BATT 3V, Q1 DMG2302UKQ-7, Q2 DMG2302UKQ-7, Q3 DMG2302UKQ-7, Q4 DMG2302UKQ-7, Q5 DMG2302UKQ-7, Q6 DMG2302UKQ-7, Q7 DMG2302UKQ-7, SW1 100SP1T1B4M2QE, SW10 100k, SW2 100SP1T1B4M2QE, SW3 100SP1T1B4M2QE, SW4 100SP1T1B4M2QE, SW5 100SP1T1B4M2QE, SW6 100SP1T1B4M2QE, SW7 100SP1T1B4M2QE, SW8 100SP1T1B4M2QE, SW9 100SP1T1B4M2QE, U1 CD74HC4017M96, U2 LMC555CMX/NOPB

Commit message: Add in changes: move to 0805 parts, routing updates
Parts:
- added J2: BATT-, Custom_Parts:SolderPad_1x1_8x8mm, B.Cu at (42.6, 115.0)
- C1, C2, C3: footprint Custom_Parts:C_0402_1005Metric -> Custom_Parts:C_0805_2012Metric
- J1: value BATT 3V -> BATT+; footprint Custom_Parts:SolderPad_1x2_10x10mm_P12.7mm -> Custom_Parts:SolderPad_1x1_8x8mm
- R11, R12, R14, R15, R3, R4, R7, R8: footprint Custom_Parts:R_0402_1005Metric -> Custom_Parts:R_0805_2012Metric
- moved C1 4.39 mm to (41.6, 107.2), turned to -90 degrees
- moved J1 3.48 mm to (33.1, 112.1)
- moved C2 2.75 mm to (41.6, 111.9), turned to 90 degrees
- moved C3 2.26 mm to (35.6, 117.2), turned to 180 degrees
- moved R15 1.17 mm to (39.7, 117.2)
- moved R11 0.25 mm to (59.1, 84.4)
- moved R12 0.25 mm to (134.2, 84.4)
- moved R14 0.25 mm to (92.2, 84.4)
- moved R3 0.25 mm to (113.2, 84.4)
- moved R4 0.25 mm to (166.2, 84.4)
- moved R7 0.25 mm to (188.2, 84.4)
- moved R8 0.25 mm to (208.2, 84.4)
Routing:
- net GND: track 25.3 -> 49.3 mm, vias 21 -> 19
- net VBAT: track 0.00 -> 21.8 mm, vias 0 -> 6
- net Net-(LED1-K): track 116.9 -> 108.8 mm
- net /Controls/TOGGLE_PWR: track 51.3 -> 56.3 mm
- net /Controls/THRESHOLD: track 18.1 -> 13.3 mm
- net LETTER_F2: track 142.9 -> 143.6 mm

Commit message: Add in final updates
Parts:
- moved SW9 21.2 mm to (42.4, 114.0)
- moved J2 17.8 mm to (31.4, 101.3)
- moved C2 11.3 mm to (41.5, 100.5)
- moved C1 10.5 mm to (41.5, 96.8)
- moved U1 10.5 mm to (37.1, 91.0)
- moved U2 10.5 mm to (37.3, 100.9)
- moved C3 10.0 mm to (35.8, 107.2)
- moved R15 10.0 mm to (39.9, 107.2)
- moved J1 9.49 mm to (40.9, 106.6), turned to 180 degrees
Connections:
- SW10 pad 1: /Controls/DISCHARGE -> unconnected-(SW10-Pad1)
- SW10 pad 3: unconnected-(SW10-Pad3) -> /Controls/DISCHARGE
Routing:
- net /Controls/THRESHOLD: track 13.3 -> 35.9 mm
- net /Controls/TOGGLE_PWR: track 56.3 -> 76.0 mm
- net /Controls/DISCHARGE: track 18.1 -> 32.4 mm
- net LETTER_F2: track 143.6 -> 137.6 mm, vias 3 -> 2
- net ALL_LETTERS: track 202.9 -> 200.3 mm, vias 14 -> 8
- net LETTER_F: track 108.9 -> 106.7 mm, vias 3 -> 2
- net LETTER_I: track 82.9 -> 81.3 mm, vias 3 -> 2
- net LETTER_R: track 58.7 -> 57.5 mm, vias 3 -> 2
- net LETTER_G: track 25.4 -> 24.2 mm
- net GND: track 49.3 -> 50.4 mm
- net LETTER_N: track 193.5 -> 193.0 mm, vias 3 -> 2
- net LETTER_I2: track 155.6 -> 156.0 mm, vias 3 -> 2
- net VBAT: track 21.8 -> 22.1 mm, vias 6 -> 9
Other:
- board text added: "Designed, assembled by Dad"
- board text added: "MINUS"
- board text added: "PLUS"
- board text added: "We love you Griffin! Love Mom, Dad, Vera"

Commit message: Add in griffin board update, this one is ordered!
Parts:
- moved H3 1.00 mm to (231.0, 76.0)
- moved H4 1.00 mm to (231.0, 134.0)
